File: schematics/on-board-controller/motor.kicad_sch (KiCad schematic)
At the start: 17 parts, among them M1 Motor_DC, M2 Motor_DC, M3 Stepper_Motor_bipolar, U1 L293D, U3 L293D

Commit message: new version, and ltspice for electromagnet
Parts:
- added D10, D11, D12, D9: LED, LED_SMD:LED_0805_2012Metric_Pad1.15x1.40mm_HandSolder, symbol Device:LED
- added R18, R19, R20, R21: 330, Resistor_SMD:R_0805_2012Metric_Pad1.20x1.40mm_HandSolder, symbol Device:R
Connections:
- net DC_MOTOR1: now also D3.2 (A); no longer D8.2 (A)
- net DC_MOTOR2: now also D4.2 (A); no longer D7.2 (A)
- net DC_MOTOR3: now also D6.2 (A); no longer D4.2 (A)
- net DC_MOTOR4: now also D7.2 (A); no longer D5.2 (A)
- net DC_MOTOR_EN1_2: now also D5.2 (A); no longer D3.2 (A)
- net DC_MOTOR_EN3_4: now also D8.2 (A); no longer D6.2 (A)
- net GND: now also R18.2, R19.2, R20.2, R21.2
- net STEPPER1: now also D9.2 (A)
- net STEPPER2: now also D10.2 (A)
- net STEPPER3: now also D11.2 (A)
- net STEPPER4: now also D12.2 (A)
- net at R12.1: now also D5.1 (K); no longer D3.1 (K)
- net at R13.1: now also D6.1 (K); no longer D4.1 (K)
- net at R14.1: now also D7.1 (K); no longer D5.1 (K)
- net at R15.1: now also D8.1 (K); no longer D6.1 (K)
- net at R17.1: now also D3.1 (K); no longer D8.1 (K)
- net at R16.1: now also D4.1 (K); no longer D7.1 (K)
- new net: D9.1 (K), R18.1
- new net: D12.1 (K), R21.1
- new net: D10.1 (K), R19.1
- new net: D11.1 (K), R20.1
Other:
- moved on the sheet: M1, M2, M3, R12, R13, R14, R15, R16, R17, U1, U3

Commit message: updated on-board schematic with changes
Parts:
- added C15, C16, C17, C18: 100n, Capacitor_SMD:C_0805_2012Metric_Pad1.18x1.45mm_HandSolder, symbol Device:C
- added C19, C20: 10u, Capacitor_THT:CP_Radial_D5.0mm_P2.50mm, symbol Device:C_Polarized
- added R23, R24: 4k7, Resistor_SMD:R_0805_2012Metric_Pad1.20x1.40mm_HandSolder, symbol Device:R
Connections:
- net +BATT: now also C17.2, C18.2, C19.1, C20.1
- net DC_MOTOR_EN1_2: now also R23.1
- net DC_MOTOR_EN3_4: now also R24.1
- net GND: now also C15.1, C16.1, C17.1, C18.1, C19.2, C20.2, R23.2, R24.2
- net +3V3 renamed +6V
- net +6V: now also C15.2, C16.2
Other:
- moved on the sheet: D10, D11, D12, D3, D4, D5, D6, D7, D8, D9, M1, M2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

Commit message: on-board: updated schematic to match STM32 confighuration
Other:
- title: sumbersible -> On-board Controller
Changed lines of the file:
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@@
 	(paper "A4")
 	(title_block
-		(title "sumbersible")
+		(title "On-board Controller")
 		(date "2024-07-16")
 		(rev "1")
