File: schematics/on-board-controller-2/mcu.kicad_sch (KiCad schematic)
At the start: 4 parts, among them J1 programmer, U4 STM32L476RGTx

Commit message: started new version
Parts:
- removed C1: 100n, Capacitor_SMD:C_0805_2012Metric_Pad1.18x1.45mm_HandSolder, symbol Device:C
- removed J1: programmer, Connector_PinSocket_2.54mm:PinSocket_1x05_P2.54mm_Vertical, symbol Connector_Generic:Conn_01x05
- removed R9: 10k, Resistor_SMD:R_0805_2012Metric_Pad1.20x1.40mm_HandSolder, symbol Device:R
- removed U4: STM32L476RGTx, Package_QFP:LQFP-64_10x10mm_P0.5mm, symbol MCU_ST_STM32L4:STM32L476RGTx
- added C10, C11, C12, C13, C14, C2, C9: 100n, Capacitor_SMD:C_0805_2012Metric_Pad1.18x1.45mm_HandSolder, symbol Device:C
- added J2: programmer, Connector_PinSocket_2.54mm:PinSocket_1x05_P2.54mm_Vertical, symbol Connector_Generic:Conn_01x05
- added R2: 10k, Resistor_SMD:R_0805_2012Metric_Pad1.20x1.40mm_HandSolder, symbol Device:R
- added U2: STM32L476RGTx, Package_QFP:LQFP-64_10x10mm_P0.5mm, symbol MCU_ST_STM32L4:STM32L476RGTx
Connections:
- net +3V3: now also C10.2, C11.2, C12.2, C13.2, C14.2, C9.2, J2.1 (Pin_1), U2.1 (VBAT), U2.13 (VDDA), U2.19 (VDD), U2.28 (PB2), U2.32 (VDD), U2.48 (VDDUSB), U2.64 (VDD)
- net GND: now also C10.1, C11.1, C12.1, C13.1, C14.1, C2.1, C9.1, J2.5 (Pin_5), R2.2, U2.12 (VSSA), U2.18 (VSS), U2.31 (VSS), U2.47 (VSS), U2.63 (VSS)
- net MISO: now also U2.56 (PB4)
- net MOSI: now also U2.57 (PB5)
- net NSS: now also U2.20 (PA4)
- net RADIO_DONE: now also U2.27 (PB1)
- net RESET: now also C2.2, J2.4 (Pin_4), U2.7 (NRST)
- net SCK: now also U2.55 (PB3)
- net SWCLK: now also J2.2 (Pin_2), U2.49 (PA14)
- net SWDIO: now also J2.3 (Pin_3), U2.46 (PA13)
- new net: R2.1, U2.60 (BOOT0)
- new net DC_MOTOR1: U2.14 (PA0)
- new net DC_MOTOR2: U2.15 (PA1)
- new net DC_MOTOR3: U2.16 (PA2)
- new net DC_MOTOR4: U2.17 (PA3)
- new net DC_MOTOR_EN1_2: U2.22 (PA6)
- new net DC_MOTOR_EN3_4: U2.23 (PA7)
- new net ELECTROMAGNET: U2.29 (PB10)
- new net RESET_RADIO: U2.26 (PB0)
- new net STEPPER1: U2.8 (PC0)
- new net STEPPER2: U2.9 (PC1)
- new net STEPPER3: U2.10 (PC2)
- new net STEPPER4: U2.11 (PC3)
- no-connect marks 24 -> 31
Other:
- title: Off-board Controller -> On-board Controller

Commit message: produced version with 2 0V floods
Connections:
- net DC_MOTOR_EN1_2: now also U2.21 (PA5); no longer U2.22 (PA6)
- net DC_MOTOR_EN3_4: now also U2.29 (PB10); no longer U2.23 (PA7)
- net ELECTROMAGNET: now also U2.55 (PB3); no longer U2.29 (PB10)
- net MISO: now also U2.35 (PB14); no longer U2.56 (PB4)
- net MOSI: now also U2.36 (PB15); no longer U2.57 (PB5)
- net NSS: now also U2.33 (PB12); no longer U2.20 (PA4)
- net SCK: now also U2.34 (PB13); no longer U2.55 (PB3)
