File: schematics/on-board-controller-2/motor.kicad_sch (KiCad schematic)
At the start: 33 parts, among them M1 Motor_DC, M2 Motor_DC, M3 Stepper_Motor_bipolar, U1 L293D, U3 L293D

Commit message: added a bom and edited layout
Parts:
- C19, C20: footprint Capacitor_THT:CP_Radial_D5.0mm_P2.50mm -> Capacitor_THT:CP_Radial_D5.0mm_P2.00mm
Changed lines of the file:
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@@
 			)
 		)
-		(property "Footprint" "Capacitor_THT:CP_Radial_D5.0mm_P2.50mm"
+		(property "Footprint" "Capacitor_THT:CP_Radial_D5.0mm_P2.00mm"
 			(at 254.9652 152.4 0)
 			(effects
@@
 			)
 		)
-		(property "Footprint" "Capacitor_THT:CP_Radial_D5.0mm_P2.50mm"
+		(property "Footprint" "Capacitor_THT:CP_Radial_D5.0mm_P2.00mm"
 			(at 267.6652 152.4 0)
 			(effects
