File: schematics/on-board-controller-2/electromagnet.kicad_sch (KiCad schematic)
At the start: 8 parts, among them Q1 NMOS

Commit message: updates
Parts:
- D13: footprint LED_SMD:LED_0805_2012Metric_Pad1.15x1.40mm_HandSolder -> Diode_THT:D_A-405_P7.62mm_Horizontal
Changed lines of the file:
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@@
 			)
 		)
-		(property "Footprint" "LED_SMD:LED_0805_2012Metric_Pad1.15x1.40mm_HandSolder"
+		(property "Footprint" "Diode_THT:D_A-405_P7.62mm_Horizontal"
 			(at 152.4 81.28 0)
 			(effects
