File: schematics/off-board-controller/mcu.kicad_sch (KiCad schematic)
At the start: 4 parts, among them J1 programmer, U4 STM32L476RGTx

Commit message: finished footprints, schematic, and started layout
Parts:
- added C4, C5, C6, C7, C8, C9: 100n, Capacitor_SMD:C_0805_2012Metric_Pad1.18x1.45mm_HandSolder, symbol Device:C
Connections:
- net +3V3: now also C4.2, C5.2, C6.2, C7.2, C8.2, C9.2
- net GND: now also C4.1, C5.1, C6.1, C7.1, C8.1, C9.1
- net TRISTATE_DOWN: now also U4.39 (PC8); no longer U4.38 (PC7)
- net TRISTATE_UP: now also U4.40 (PC9); no longer U4.39 (PC8)
- net CS_IO1-2: now reaches U4.14 (PA0)
- net CS_IO3-4: now reaches U4.15 (PA1)
- net CS_RADIO: now reaches U4.16 (PA2)
- net 7SEG_D1: no longer names the net of U4.33 (PB12)
- net 7SEG_D2: no longer names the net of U4.34 (PB13)
- net 7SEG_D3: no longer names the net of U4.35 (PB14)
- net 7SEG_D4: no longer names the net of U4.36 (PB15)
- net 7SEG_DP: no longer names the net of U4.62 (PB9)
- net 7SEG_a: no longer names the net of U4.26 (PB0)
- net 7SEG_b: no longer names the net of U4.27 (PB1)
- net 7SEG_c: no longer names the net of U4.28 (PB2)
- net 7SEG_d: no longer names the net of U4.57 (PB5)
- net 7SEG_e: no longer names the net of U4.58 (PB6)
- net 7SEG_f: no longer names the net of U4.59 (PB7)
- net 7SEG_g: no longer names the net of U4.61 (PB8)
- net NSS: no longer names the net of U4.20 (PA4)
- net RADIO_RESET renamed RESET_IO
- no-connect marks 24 -> 34

Commit message: produced first draft of layout design
Connections:
- net +3V3: now also U4.28 (PB2)
- no-connect marks 34 -> 33
Changed lines of the file:
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@@
-	)
-	(no_connect
-		(at 143.51 101.6)
 	)
 	(no_connect
@@
 	(wire
 		(pts
+			(xy 151.13 101.6) (xy 151.13 99.06)
+		)
+		(stroke
+			(width 0)
+			(type default)
+		)
+	)
+	(wire
+		(pts
 			(xy 204.47 43.18) (xy 219.71 43.18)
 		)
@@
 		(pts
 			(xy 219.71 43.18) (xy 234.95 43.18)
+		)
+		(stroke
+			(width 0)
+			(type default)
+		)
+	)
+	(wire
+		(pts
+			(xy 143.51 101.6) (xy 151.13 101.6)
 		)
 		(stroke
@@
 					(unit 1)
 				)
+			)
+		)
+	)
+	(symbol
+		(lib_id "power:+3V3")
+		(at 151.13 99.06 0)
+		(unit 1)
+		(exclude_from_sim no)
+		(in_bom yes)
+		(on_board yes)
+		(dnp no)
+		(fields_autoplaced yes)
+		(property "Reference" "#PWR04"
+			(at 151.13 102.87 0)
+			(effects
+				(font
+					(size 1.27 1.27)
+				)
+				(hide yes)
+			)
+		)
+		(property "Value" "+3V3"
+			(at 151.13 93.98 0)
+			(effects
+				(font
+					(size 1.27 1.27)
+				)
+			)
+		)
+		(property "Footprint" ""
+			(at 151.13 99.06 0)
+			(effects
+				(font
+					(size 1.27 1.27)
+				)
+				(hide yes)
+			)
+		)
+		(property "Datasheet" ""
+			(at 151.13 99.06 0)
+			(effects
+				(font
+					(size 1.27 1.27)
+				)
+				(hide yes)
+			)
+		)
+		(property "Description" "Power symbol creates a global label with name \"+3V3\""
+			(at 151.13 99.06 0)
+			(effects
+				(font
+					(size 1.27 1.27)
+				)
+				(hide yes)
+			)
+		)
+		(pin "1"
+		)
+		(instances
+			(project "controller"
+				(path "/0775f04a-8a0e-41f5-b442-dacb2efdb863/91cafd9f-69c3-4236-80de-a9ef98ffb65d"
+					(reference "#PWR04")
+					(unit 1)
+				)
