File: schematics/off-board-controller/controller.kicad_pcb (KiCad board)
At the start: 2 copper layers, 80 x 90 mm, 70 parts, among them J1 programmer, J2 5-1814832-1, J3 9V, SW5 SW_SPDT_MSM, U4 STM32L476RGTx, U5 RFM98W-433S2, U6 L78L33_TO92, U8 MCP23S17_SP, U9 MCP23S17_SP

Commit message: updated footprints for through hole components with long legs
Parts:
- moved U6 0.31 mm to (160.5, 126.4)
Changed lines of the file:
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@@
 	(footprint "Package_TO_SOT_THT:TO-92_Inline"
 		(layer "F.Cu")
-		(at 160.185 126.445 -90)
+		(at 160.5 126.445 -90)
 		(descr "TO-92 leads in-line, narrow, oval pads, drill 0.75mm (see NXP sot054_po.pdf)")
 		(tags "to-92 sc-43 sc-43a sot54 PA33 transistor")
@@
 			(at -2.445 -2.315 90)
 			(layer "F.SilkS")
+			(hide yes)
 			(effects
 				(font
@@
 			(at 1.27 2.79 90)
 			(layer "F.Fab")
+			(hide yes)
 			(effects
 				(font
@@
 			)
 		)
+		(property "Sim.Device" "NMOS"
+			(at 0 0 -90)
+			(unlocked yes)
+			(layer "F.Fab")
+			(hide yes)
+			(effects
+				(font
+					(size 1 1)
+					(thickness 0.15)
+				)
+			)
+		)
+		(property "Sim.Pins" "1=D 2=G 3=S"
+			(at 0 0 -90)
+			(unlocked yes)
+			(layer "F.Fab")
+			(hide yes)
+			(effects
+				(font
+					(size 1 1)
+					(thickness 0.15)
+				)
+			)
+		)
+		(property "Sim.Type" "VDMOS"
+			(at 0 0 -90)
+			(unlocked yes)
+			(layer "F.Fab")
+			(hide yes)
+			(effects
+				(font
+					(size 1 1)
+					(thickness 0.15)
+				)
+			)
+		)
+		(property "Sim.Pins" "1=D 2=G 3=S"
+			(at 0.004375 0.123375 -90)
+			(unlocked yes)
+			(layer "F.Fab")
+			(hide yes)
+			(effects
+				(font
+					(size 1 1)
+					(thickness 0.15)
+				)
+			)
+		)
+		(property "Sim.Type" "VDMOS"
+			(at 0.329 0.121 -90)
+			(unlocked yes)
+			(layer "F.Fab")
+			(hide yes)
+			(effects
+				(font
+					(size 1 1)
+					(thickness 0.15)
+				)
+			)
+		)
+		(property "Sim.Device" "NMOS"
+			(at 0.004375 0.123375 -90)
+			(unlocked yes)
+			(layer "F.Fab")
+			(hide yes)
+			(effects
+				(font
+					(size 1 1)
+					(thickness 0.15)
+				)
+			)
+		)
 		(property ki_fp_filters "TO?92*")
 		(sheetname "power")
@@
 		(attr through_hole)
 		(fp_line
-			(start -0.53 1.85)
-			(end 3.07 1.85)
+			(start -0.201 1.971)
+			(end 3.734391 1.959478)
 			(stroke
 				(width 0.12)
@@
 		)
 		(fp_arc
-			(start -0.568478 1.838478)
-			(mid -1.132087 -0.994977)
-			(end 1.27 -2.6)
+			(start -0.251426 1.971426)
+			(mid -0.757888 -1.016203)
+			(end 1.895913 -2.479)
 			(stroke
 				(width 0.12)
@@
 		)
 		(fp_arc
-			(start 1.27 -2.6)
-			(mid 3.672087 -0.994977)
-			(end 3.108478 1.838478)
+			(start 1.895913 -2.479)
+			(mid 4.298005 -0.873976)
+			(end 3.734391 1.959478)
 			(stroke
 				(width 0.12)
@@
 		)
 		(fp_line
-			(start 4 2.01)
-			(end -1.46 2.01)
+			(start 4.647 2.131)
+			(end -1.131 2.131)
 			(stroke
 				(width 0.05)
@@
 		)
 		(fp_line
-			(start 4 2.01)
-			(end 4 -2.73)
+			(start 4.647 2.131)
+			(end 4.647 -2.609)
 			(stroke
 				(width 0.05)
@@
 		)
 		(fp_line
-			(start -1.46 -2.73)
-			(end -1.46 2.01)
+			(start -1.131 -2.609)
+			(end -1.131 2.131)
 			(stroke
 				(width 0.05)
@@
 		)
 		(fp_line
-			(start -1.46 -2.73)
-			(end 4 -2.73)
+			(start -1.131 -2.609)
+			(end 4.647 -2.609)
 			(stroke
 				(width 0.05)
@@
 		)
 		(fp_line
-			(start -0.5 1.75)
-			(end 3 1.75)
+			(start -0.197013 2.001775)
+			(end 3.734391 1.959478)
 			(stroke
 				(width 0.1)
@@
 		)
 		(fp_arc
-			(start -0.483625 1.753625)
-			(mid -1.021221 -0.949055)
-			(end 1.27 -2.48)
+			(start -0.263632 1.983632)
+			(mid -0.749039 -1.072946)
+			(end 2.006779 -2.481405)
 			(stroke
 				(width 0.1)
@@
 		)
 		(fp_arc
-			(start 1.27 -2.48)
-			(mid 3.561221 -0.949055)
-			(end 3.023625 1.753625)
+			(start 2.006779 -2.481405)
+			(mid 4.389324 -0.85179)
+			(end 3.734391 1.959478)
 			(stroke
 				(width 0.1)
@@
 		)
 		(fp_text user "${REFERENCE}"
-			(at 1.27 0 90)
+			(at 1.274375 0.123375 90)
 			(layer "F.Fab")
 			(effects
@@
 		)
 		(pad "1" thru_hole rect
-			(at 0 0 270)
-			(size 1.05 1.5)
+			(at 0 0.127 270)
+			(size 1.3 1.5)
 			(drill 0.75)
 			(layers "*.Cu" "*.Mask")
@@
 		)
 		(pad "2" thru_hole oval
-			(at 1.27 0 270)
-			(size 1.05 1.5)
+			(at 1.778 0.127 270)
+			(size 1.3 1.5)
 			(drill 0.75)
 			(layers "*.Cu" "*.Mask")
@@
 		)
 		(pad "3" thru_hole oval
-			(at 2.54 0 270)
-			(size 1.05 1.5)
+			(at 3.556 0.127 270)
+			(size 1.3 1.5)
 			(drill 0.75)
 			(layers "*.Cu" "*.Mask")
@@
 	)
 	(via
-		(at 160 132)
+		(at 160.25 131.75)
 		(size 0.6)
 		(drill 0.3)
@@
 	)
 	(segment
-		(start 158.3 130.87)
-		(end 160.185 128.985)
+		(start 157.185 130.87)
+		(end 159.504 130.87)
 		(width 0.5)
 		(layer "F.Cu")
@@
 	)
 	(segment
-		(start 164.705 128.985)
-		(end 167 126.69)
+		(start 160.624 129.75)
+		(end 163.94 129.75)
 		(width 0.5)
 		(layer "F.Cu")
@@
 	)
 	(segment
-		(start 160.185 128.985)
-		(end 164.705 128.985)
+		(start 159.504 130.87)
+		(end 160.624 129.75)
 		(width 0.5)
 		(layer "F.Cu")
@@
 	)
 	(segment
-		(start 157.185 130.87)
-		(end 158.3 130.87)
+		(start 163.94 129.75)
+		(end 167 126.69)
 		(width 0.5)
 		(layer "F.Cu")
@@
 	)
 	(segment
+		(start 158.185 126.445)
+		(end 157.185 125.445)
+		(width 0.5)
+		(layer "F.Cu")
+		(net 4)
+	)
+	(segment
 		(start 149.5 59.25)
 		(end 151 60.75)
@@
 	)
 	(segment
+		(start 160.373 126.445)
+		(end 158.185 126.445)
+		(width 0.5)
+		(layer "F.Cu")
+		(net 4)
+	)
+	(segment
 		(start 157.185 118.355)
 		(end 157.045 118.215)
@@
 	)
 	(segment
-		(start 158.185 126.445)
-		(end 157.185 125.445)
-		(width 0.5)
-		(layer "F.Cu")
-		(net 4)
-	)
-	(segment
 		(start 134.75 50)
 		(end 144 59.25)
@@
 		(width 0.5)
 		(layer "F.Cu")
-		(net 4)
-	)
-	(segment
-		(start 160.185 126.445)
-		(end 158.185 126.445)
-		(width 0.5)
-		(layer "F.Cu")
